Commit message: tem que ver os launch files

File: src/description/complete-bot-description.urdf (robot description, URDF)
Before this commit: robot complete_bot, 7 links, 6 joints
Joints:
- removed joint lidar_joint
- added joint lidar_joint_${namespace}: type fixed, parent base_link, child lidar_link, origin xyz=0 0 ${base_height/2+0.01} rpy=0 0 0

Commit message: launch files funcionando

File: src/description/complete-bot-description.urdf (robot description, URDF)
Before this commit: robot complete_bot, 7 links, 6 joints
Joints:
- removed joint lidar_joint_${namespace}
- added joint lidar_joint: type fixed, parent base_link, child lidar_link, origin xyz=0 0 ${base_height/2+0.01} rpy=0 0 0

Commit message: transformacoes ok

File: src/description/complete-bot-description.urdf (robot description, URDF)
Before this commit: robot complete_bot, 7 links, 6 joints
Links:
- removed link base_footprint
- removed link base_link
- removed link camera_depth_frame
- removed link camera_link
- removed link front_caster
- removed link imu_link
- removed link lidar_link
- added link $(arg namespace)_base_footprint
- added link $(arg namespace)_base_link; collision cylinder length=${base_height} radius=${base_radius}; visual cylinder length=${base_height} radius=${base_radius}
- added link $(arg namespace)_camera_depth_frame
- added link $(arg namespace)_camera_link, mass 0.035; collision box size=0.015 0.130 0.022; visual box size=0.015 0.130 0.022
- added link $(arg namespace)_front_caster; collision sphere radius=${(wheel_radius+wheel_zoff-(base_height/2))}; visual sphere radius=${(wheel_radius+wheel_zoff-(base_height/2))}
- added link $(arg namespace)_imu_link; collision box size=0.1 0.1 0.1; visual box size=0.1 0.1 0.1
- added link $(arg namespace)_lidar_link, mass 0.125; collision cylinder length=0.055 radius=0.0508; visual cylinder length=0.055 radius=0.0508
Joints:
- removed joint base_joint
- removed joint camera_depth_joint
- removed joint camera_joint
- removed joint caster_joint
- removed joint imu_joint
- removed joint lidar_joint
- added joint $(arg namespace)_base_joint: type fixed, parent $(arg namespace)_base_link, child $(arg namespace)_base_footprint, origin xyz=0.0 0.0 ${-(wheel_radius+wheel_zoff)} rpy=0 0 0
- added joint $(arg namespace)_camera_depth_joint: type fixed, parent $(arg namespace)_camera_link, child $(arg namespace)_camera_depth_frame, origin xyz=0 0 0 rpy=${-pi/2} 0 ${-pi/2}
- added joint $(arg namespace)_camera_joint: type fixed, parent $(arg namespace)_base_link, child $(arg namespace)_camera_link, origin xyz=${base_radius} 0 0.05 rpy=0 0 0
- added joint $(arg namespace)_caster_joint: type fixed, parent $(arg namespace)_base_link, child $(arg namespace)_front_caster, origin xyz=${caster_xoff} 0.0 ${-(base_height/2)} rpy=0 0 0
- added joint $(arg namespace)_imu_joint: type fixed, parent $(arg namespace)_base_link, child $(arg namespace)_imu_link, origin xyz=0 0 0.01
- added joint $(arg namespace)_lidar_joint: type fixed, parent $(arg namespace)_base_link, child $(arg namespace)_lidar_link, origin xyz=0 0 ${base_height/2+0.01} rpy=0 0 0

File: src/description/rl-bot-description.urdf (robot description, URDF)
Before this commit: robot complete_bot, 5 links, 4 joints
Links:
- removed link base_footprint
- removed link base_link
- removed link front_caster
- removed link imu_link
- removed link lidar_link
- added link $(arg namespace)_base_footprint
- added link $(arg namespace)_base_link; collision cylinder length=${base_height} radius=${base_radius}; visual cylinder length=${base_height} radius=${base_radius}
- added link $(arg namespace)_front_caster; collision sphere radius=${(wheel_radius+wheel_zoff-(base_height/2))}; visual sphere radius=${(wheel_radius+wheel_zoff-(base_height/2))}
- added link $(arg namespace)_imu_link; collision box size=0.1 0.1 0.1; visual box size=0.1 0.1 0.1
- added link $(arg namespace)_lidar_link, mass 0.125; collision cylinder length=0.055 radius=0.0508; visual cylinder length=0.055 radius=0.0508
Joints:
- removed joint base_joint
- removed joint caster_joint
- removed joint imu_joint
- removed joint lidar_joint
- added joint $(arg namespace)_base_joint: type fixed, parent $(arg namespace)_base_link, child $(arg namespace)_base_footprint, origin xyz=0.0 0.0 ${-(wheel_radius+wheel_zoff)} rpy=0 0 0
- added joint $(arg namespace)_caster_joint: type fixed, parent $(arg namespace)_base_link, child $(arg namespace)_front_caster, origin xyz=${caster_xoff} 0.0 ${-(base_height/2)} rpy=0 0 0
- added joint $(arg namespace)_imu_joint: type fixed, parent $(arg namespace)_base_link, child $(arg namespace)_imu_link, origin xyz=0 0 0.01
- added joint $(arg namespace)_lidar_joint: type fixed, parent $(arg namespace)_base_link, child $(arg namespace)_lidar_link, origin xyz=0 0 ${base_height/2+0.01} rpy=0 0 0

Commit message: robo andando e nao cai para o infinito

File: src/description/complete-bot-description.urdf (robot description, URDF)
Before this commit: robot complete_bot, 7 links, 6 joints
Links:
- removed link $(arg namespace)_imu_link
- link $(arg namespace)_base_link: geometry collision box size=${base_length} ${base_width} ${base_height}; visual box size=${base_length} ${base_width} ${base_height}
Joints:
- removed joint $(arg namespace)_imu_joint
- joint $(arg namespace)_camera_joint: origin xyz=${base_radius} 0 0.05 rpy=0 0 0 -> xyz=${base_length/2} 0 0.01 rpy=0 0 0
- joint $(arg namespace)_caster_joint: type fixed -> continuous

File: src/description/rl-bot-description.urdf (robot description, URDF)
Before this commit: robot complete_bot, 5 links, 4 joints
Links:
- removed link $(arg namespace)_imu_link
- link $(arg namespace)_base_link: geometry collision box size=${base_length} ${base_width} ${base_height}; visual box size=${base_length} ${base_width} ${base_height}
Joints:
- removed joint $(arg namespace)_imu_joint
- joint $(arg namespace)_caster_joint: type fixed -> continuous

Commit message: deteccao de imagem comcliuda

File: src/description/complete-bot-description.urdf (robot description, URDF)
Before this commit: robot complete_bot, 6 links, 5 joints
Links:
- removed link $(arg namespace)_base_footprint
- removed link $(arg namespace)_base_link
- removed link $(arg namespace)_camera_depth_frame
- removed link $(arg namespace)_camera_link
- removed link $(arg namespace)_front_caster
- removed link $(arg namespace)_lidar_link
- added link base_footprint
- added link base_link; collision box size=${base_length} ${base_width} ${base_height}; visual box size=${base_length} ${base_width} ${base_height}
- added link camera_depth_frame
- added link camera_link, mass 0.035; collision box size=0 0 0; visual box size=0 0 0
- added link front_caster; collision sphere radius=${(wheel_radius+wheel_zoff-(base_height/2))}; visual sphere radius=${(wheel_radius+wheel_zoff-(base_height/2))}
- added link lidar_link, mass 0.125; collision cylinder length=0.055 radius=0.0508; visual cylinder length=0.055 radius=0.0508
Joints:
- removed joint $(arg namespace)_base_joint
- removed joint $(arg namespace)_camera_depth_joint
- removed joint $(arg namespace)_camera_joint
- removed joint $(arg namespace)_caster_joint
- removed joint $(arg namespace)_lidar_joint
- added joint base_joint: type fixed, parent base_link, child base_footprint, origin xyz=0.0 0.0 ${-(wheel_radius+wheel_zoff)} rpy=0 0 0
- added joint camera_depth_joint: type fixed, parent camera_link, child camera_depth_frame, origin xyz=1 1 1 rpy=${-pi/2} 0 ${-pi/2}
- added joint camera_joint: type fixed, parent base_link, child camera_link, origin xyz=${base_length/2} 0 0.01 rpy=0 0 0
- added joint caster_joint: type continuous, parent base_link, child front_caster, origin xyz=${caster_xoff} 0.0 ${-(base_height/2)} rpy=0 0 0
- added joint lidar_joint: type fixed, parent base_link, child lidar_link, origin xyz=0 0 ${base_height/2+0.01} rpy=0 0 0
