Commit message: perfeitamente funcional para launch mono robot, tem suporte para namespace mas ainda nao funciona direito

File: src/description/rl-bot-description.urdf (robot description, URDF)
Before this commit: robot rl_bot, 4 links, 3 joints
Links:
- removed link $(arg namespace)_base_footprint
- removed link $(arg namespace)_base_link
- removed link $(arg namespace)_front_caster
- removed link $(arg namespace)_lidar_link
- added link base_footprint
- added link base_link; collision box size=${base_length} ${base_width} ${base_height}; visual box size=${base_length} ${base_width} ${base_height}
- added link front_caster; collision sphere radius=${(wheel_radius+wheel_zoff-(base_height/2))}; visual sphere radius=${(wheel_radius+wheel_zoff-(base_height/2))}
- added link lidar_link, mass 0.125; collision cylinder length=0.055 radius=0.0508; visual cylinder length=0.055 radius=0.0508
Joints:
- removed joint $(arg namespace)_base_joint
- removed joint $(arg namespace)_caster_joint
- removed joint $(arg namespace)_lidar_joint
- added joint base_joint: type fixed, parent base_link, child base_footprint, origin xyz=0.0 0.0 ${-(wheel_radius+wheel_zoff)} rpy=0 0 0
- added joint caster_joint: type continuous, parent base_link, child front_caster, origin xyz=${caster_xoff} 0.0 ${-(base_height/2)} rpy=0 0 0
- added joint lidar_joint: type fixed, parent base_link, child lidar_link, origin xyz=0 0 ${base_height/2+0.01} rpy=0 0 0
